File: hardware/kicad/vectra-auto-lights.kicad_sch (KiCad schematic)
At the start: 48 parts, among them J1 KL30+GND, J2 CAR_INPUTS, J3 J_XENON, J4 J_GABARI, J5 J_FOG, J6 J_ILLUM, K1 Relay_12V, K2 Relay_12V, Q1 IRF4905, Q2 2N7000, Q3 BC547, Q4 BC547, Q5 BC547, U1 ESP32_DevKit_v1, U2 LM7805

Commit message: Fix KiCad 10 compatibility: remove invalid syntax, fix library names
PCB (.kicad_pcb):
- Remove all ;; comments (not valid in S-expression format)
- Replace incomplete footprint stubs with proper mounting hole pads
- Keep board outline 120x80mm + GND pour; components added via
  Tools -> Update PCB from Schematic

Schematic (.kicad_sch):
- Opto:PC817 -> Isolator:PC817 (library renamed in KiCad 8+)
- Relay:G5V-2 (DPDT) -> Relay:G5V-1 (SPDT, correct for K1/K2)
- Regenerate vectra-auto-lights.kicad_sch

Co-Authored-By: Claude Sonnet 4.6 <noreply@anthropic.com>
Parts:
- removed K1, K2: Relay_12V, Relay_THT:Relay_SPDT_Omron_G5V-2, symbol Relay:G5V-2
- removed OK1, OK2, OK3: PC817, Package_DIP:DIP-4_W7.62mm, symbol Opto:PC817
- added K1, K2: Relay_12V, Relay_THT:Relay_SPDT_Omron_G5V-1, symbol Relay:G5V-1
- added OK1, OK2, OK3: PC817, Package_DIP:DIP-4_W7.62mm, symbol Isolator:PC817
Changed lines of the file:
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@@
     (effects (font (size 1.27 1.27)) (justify left))
   )
-  (symbol (lib_id "Opto:PC817") (at 58.0000 118.0000 0) (unit 1)
+  (symbol (lib_id "Isolator:PC817") (at 58.0000 118.0000 0) (unit 1)
     (exclude_from_sim no) (in_bom yes) (on_board yes)
     (property "Reference" "OK1" (at 59.0000 115.4600 0)
@@
     (effects (font (size 1.27 1.27)) (justify left))
   )
-  (symbol (lib_id "Opto:PC817") (at 58.0000 143.0000 0) (unit 1)
+  (symbol (lib_id "Isolator:PC817") (at 58.0000 143.0000 0) (unit 1)
     (exclude_from_sim no) (in_bom yes) (on_board yes)
     (property "Reference" "OK2" (at 59.0000 140.4600 0)
@@
     (effects (font (size 1.27 1.27)) (justify left))
   )
-  (symbol (lib_id "Opto:PC817") (at 58.0000 168.0000 0) (unit 1)
+  (symbol (lib_id "Isolator:PC817") (at 58.0000 168.0000 0) (unit 1)
     (exclude_from_sim no) (in_bom yes) (on_board yes)
     (property "Reference" "OK3" (at 59.0000 165.4600 0)
@@
     (effects (font (size 1.27 1.27)) (justify left))
   )
-  (symbol (lib_id "Relay:G5V-2") (at 270.0000 90.0000 0) (unit 1)
+  (symbol (lib_id "Relay:G5V-1") (at 270.0000 90.0000 0) (unit 1)
     (exclude_from_sim no) (in_bom yes) (on_board yes)
     (property "Reference" "K1" (at 271.0000 87.4600 0)
@@
       (effects (font (size 1.27 1.27)))
     )
-    (property "Footprint" "Relay_THT:Relay_SPDT_Omron_G5V-2" (at 270.0000 90.0000 0)
+    (property "Footprint" "Relay_THT:Relay_SPDT_Omron_G5V-1" (at 270.0000 90.0000 0)
       (effects (font (size 1.27 1.27)) hide)
     )
@@
     (effects (font (size 1.27 1.27)) (justify left))
   )
-  (symbol (lib_id "Relay:G5V-2") (at 270.0000 130.0000 0) (unit 1)
+  (symbol (lib_id "Relay:G5V-1") (at 270.0000 130.0000 0) (unit 1)
     (exclude_from_sim no) (in_bom yes) (on_board yes)
     (property "Reference" "K2" (at 271.0000 127.4600 0)
@@
       (effects (font (size 1.27 1.27)))
     )
-    (property "Footprint" "Relay_THT:Relay_SPDT_Omron_G5V-2" (at 270.0000 130.0000 0)
-      (effects (font (size 1.27 1.27)) hide)
-    )
+    (property "Footprint" "Relay_THT:Relay_SPDT_Omron_G5V-1" (at 270.0000 130.0000 0)
+      (effects (font (size 1.27 1.27)) hide)
+    )
